File: TrackingServo.kicad_sch (KiCad schematic)
At the start: 0 parts

Commit message: cleaned up schematic
Parts:
- added C1, C3, C4: 10n, symbol Device:C
- added C10, C11, C12, C2, C8: 100n, symbol Device:C
- added C5, C9: 22n, symbol Device:C
- added D1, D2, D3, D4, D5: 1N4148, symbol Device:D
- added LD1: D_Laser_1C2A, symbol Device:D_Laser_1C2A
- added M1: MOTOR, symbol Motor:Motor_DC
- added Q1, Q3, Q4: NPN, symbol Simulation_SPICE:NPN
- added Q5, Q7: 2N4401, symbol Simulation_SPICE:NPN
- added Q6: 2N7000, symbol Device:Q_NMOS_SGD
- added R1, R48, R8: 100k, symbol Device:R_US
- added R10, R11, R7: 470, symbol Device:R_US
- added R12, R13, R14, R18, R24, R25, R3, R37, R38, R39, R40, R41, R43, R44, R47: 10k, symbol Device:R_US
- added R15: 1k8, symbol Device:R_US
- added R16: 4k7, symbol Device:R_US
- added R19, R21, R22, R23, R5, R51, R54, R55, R9: 1k, symbol Device:R_US
- added R2, R49: 1M, symbol Device:R_US
- added R35: 100, symbol Device:R_US
- added R36: 390, symbol Device:R_US
- added R4: 150k, symbol Device:R_US
- added R45: 3k3, symbol Device:R_US
- added R46: 22k, symbol Device:R_US
- added R50: 2k2, symbol Device:R_US
- added R6: 47k, symbol Device:R_US
- added RV1, RV5, RV6, RV7: 100k, symbol Device:R_Potentiometer_US
- added RV3: 10k, symbol Device:R_Potentiometer_US
- added RV8: 30k, symbol Device:R_Potentiometer_US
- added SC1: Solar Cell, symbol Device:Solar_Cell
- added SW3: LEFT, symbol Switch:SW_Push
- added SW4: RIGHT, symbol Switch:SW_Push
- added U12 (x2), U18, U25, U6: 4001, symbol 4xxx:4001
- added U14, U16, U3: LM324, symbol Amplifier_Operational:LM324
- added U15: NE555P, Package_DIP:DIP-8_W7.62mm, symbol Timer:NE555P
- added U17, U19: ${SIM.PARAMS}, symbol Simulation_SPICE:OPAMP
- added U2, U22, U5: LM339, symbol Comparator:LM339
- added U21, U9: 4066, symbol 4xxx:4066
- added U23: L293D, Package_DIP:DIP-16_W7.62mm, symbol Driver_Motor:L293D
- added U4: LM555xN, Package_DIP:DIP-8_W7.62mm, symbol Timer:LM555xN
- added U7: 40106, symbol 4xxx:40106
Connections:
- new net: R43.1, U18.3, U6.5
- new net: U12.1, U12.2, U9.4
- new net: U12.3, U9.5
- new net: R46.2, R47.1, U19.2 (-)
- new net: Q6.2 (G), R49.2, R50.2, U22.2, U23.7 (2A)
- new net: R14.1, R18.2, U21.8, U22.4 (-), U9.8
- new net: R48.2, R49.1, U22.5 (+)
- new net: C8.2, D2.1 (K), R41.1, U19.1 (+)
- new net: D2.2 (A), U17.5
- new net: C1.1, SC1.1 (+)
- new net: C1.2, R2.1, R3.1, U3.3 (+)
- new net: D3.1 (K), U21.6
- new net: R19.1, R25.1, SW4.1, U25.1
- new net: Q3.2 (B), R24.1, SW3.1, U25.2
- new net: R54.2, U25.3
- new net: U18.1, U2.2
- new net: U18.2, U6.4
- new net: C5.1, C8.1, Q1.3 (E), R35.2, U15.2 (TR), U15.6 (THR)
- new net: C3.1, U15.5 (CV)
- new net: R35.1, U15.7 (DIS)
- new net: R9.2, U5.5 (+)
- new net: R5.2, R6.1, U4.7 (DIS)
- new net: R10.1, RV3.3, U5.4 (-)
- new net: R39.1, R45.2, U14.1, U14.2 (-)
- new net: R12.2, R13.1, U14.3 (+)
- new net: C4.1, R6.2, U4.2 (TR), U4.6 (THR)
- new net: D5.2 (A), Q4.1 (C), R23.1
- new net: Q4.2 (B), R22.1
- new net: R2.2, RV1.2
- new net: RV7.2, U5.6 (-)
- new net: U12.3, U9.6
- new net: C9.1, U17.1 (+)
- new net: R41.2, U17.2 (-)
- new net: Q1.1 (C), R36.1
- new net: Q1.2 (B), R15.1, R16.2
- new net: U5.1, U6.6
- new net: R38.1, U16.1, U16.2 (-)
- new net: RV5.2, U16.3 (+)
- new net: R37.1, U14.6 (-), U14.7
- new net: R37.2, R40.1, U14.13 (-)
- new net: R46.1, R48.1, U19.5
- new net: D3.2 (A), Q7.1 (C), R55.1, U12.1, U12.2
- new net: C12.1, M1.1 (+), U23.3 (1Y)
- new net: C12.2, M1.2 (-), U23.6 (2Y)
- new net: R44.2, R45.1, U14.9 (-)
- new net: RV6.2, U2.4 (-)
- new net: R1.2, RV1.1
- new net: R11.2, U5.2, U7.1
- new net: RV8.2, U2.5 (+), U5.7 (+)
- new net: Q6.3 (D), R51.2, U23.2 (1A)
- new net: Q5.2 (B), R19.2
- new net: Q3.1 (C), R21.1, R22.2
- new net: R40.2, U14.10 (+), U14.14
- new net: R38.2, R39.2, U14.12 (+)
- new net: D4.2 (A), Q5.3 (E)
- new net: LD1.2 (A), U4.3 (Q)
- new net: Q7.2 (B), R54.1
- new net: D1.2 (A), R4.1, U3.1
- new net: R4.2, R7.1, U3.2 (-)
- new net +15V: C11.1, R11.1, R12.1, R14.2, R15.2, R21.2, R23.2, R36.2, R55.2, RV5.1, RV6.1, RV7.1, RV8.1, U15.4 (R), U15.8 (VCC), U17.4 (V-), U19.3 (V+), U23.8 (VCC2)
- new net +5V: C10.1, R1.1, R5.1, R50.1, R51.1, RV3.1, RV3.2, SW3.2, SW4.2, U23.1 (EN1,2), U23.16 (VCC1), U4.4 (R), U4.8 (VCC)
- new net CLOSED_LOOP: R44.1, U14.8, U9.9
- new net GND: C10.2, C11.2, C2.1, C3.2, C4.2, C5.2, C9.2, D4.1 (K), LD1.1 (K), Q3.3 (E), Q4.3 (E), Q6.1 (S), Q7.3 (E), R10.2, R13.2, R16.1, R18.1, R24.2, R25.2, R3.2, R47.2, R7.2, R8.1, RV1.3, RV5.3, RV6.3, RV7.3, RV8.3, SC1.2 (-), U15.1 (GND), U17.3 (V+), U19.4 (V-), U23.12 (GND), U23.13 (GND), U23.4 (GND), U23.5 (GND), U4.1 (GND)
- new net LOCK: U7.2, U9.3
- new net SCANNING: D5.1 (K), Q5.1 (C), R43.2, U21.9
- new net SOLAR_POS: C2.2, D1.1 (K), R8.2, R9.1, U14.5 (+)
Other:
- removed sheet Feedback Controller
- removed sheet Laser Driver
- removed sheet Motor Driver
- removed sheet Solar Cell Frontend
- removed sheet State Machine
- note added: "P Control"
- note added: "Sweeping Mode"
